File: thingy.brd (EAGLE design)
At the start: 20 parts, among them IC1 MCP6001T-I/OT, IC2 MAX9812LEXT+T, IC3 ESP-12, IC4 ADXL345BCCZ, J1 Interface, Q1 Electret Mic

Commit message: foo
Parts:
- added J2: GPIO, pinhead:1X04
- added J3: Interrupts, pinhead:1X02
- added R10, R11: 4.7kΩ, freetronics-luke:0603
Connections:
- removed net !ACC_CS: IC3.GPIO16, IC4.7
- removed net MISO: IC3.GPIO12, IC4.12
- removed net MOSI: IC3.GPIO13, IC4.13
- removed net SCK: IC3.GPIO14, IC4.14
- new net GPIO12: IC3.GPIO12, J2.1
- new net GPIO13: IC3.GPIO13, J2.2
- new net GPIO14: IC3.GPIO14, J2.3
- new net GPIO16: IC3.GPIO16, J2.4
- new net SCL: IC3.GPIO5, IC4.14, R11.1
- new net SDA: IC3.GPIO4, IC4.13, R10.1
- net +3.3V: now also IC4.12, IC4.7, R10.2, R11.2
- net ACC_INT1: now also J3.1; no longer IC3.GPIO4
- net ACC_INT2: now also J3.2; no longer IC3.GPIO5
Changed lines of the file:
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@@
 <attribute name="PACKAGE" value="0603" x="15.5178125" y="35.1234375" size="0.4064" layer="27" display="off"/>
+</element>
+<element name="J3" library="pinhead" package="1X02" value="Interrupts" x="57.785" y="10.874375" rot="R90"/>
+<element name="J2" library="pinhead" package="1X04" value="GPIO" x="52.784375" y="11.90625" rot="R90"/>
+<element name="R11" library="freetronics-luke" package="0603" value="4.7kΩ" x="23.098125" y="34.8853125">
+<attribute name="PACKAGE" value="0603" x="23.098125" y="34.8853125" size="0.4064" layer="27" display="off"/>
+</element>
+<element name="R10" library="freetronics-luke" package="0603" value="4.7kΩ" x="23.574375" y="38.338125">
+<attribute name="PACKAGE" value="0603" x="23.574375" y="38.338125" size="0.4064" layer="27" display="off"/>
 </element>
 </elements>
@@
 <contactref element="R9" pad="2"/>
 <contactref element="R2" pad="2"/>
+<contactref element="IC4" pad="12"/>
+<contactref element="IC4" pad="7"/>
+<contactref element="R10" pad="2"/>
+<contactref element="R11" pad="2"/>
 <wire x1="22.2959375" y1="6.4290625" x2="46.4740625" y2="8.41375" width="0" layer="19" extent="1-1"/>
-<wire x1="14.8940625" y1="5.540625" x2="22.2959375" y2="6.4290625" width="0" layer="19" extent="1-1"/>
-<wire x1="14.8940625" y1="9.540625" x2="14.8940625" y2="5.540625" width="0" layer="19" extent="1-1"/>
+<wire x1="17.0940625" y1="8.740625" x2="22.2959375" y2="6.4290625" width="0" layer="19" extent="1-1"/>
+<wire x1="14.8940625" y1="9.540625" x2="17.0940625" y2="8.740625" width="0" layer="19" extent="1-1"/>
+<wire x1="15.9940625" y1="5.440625" x2="17.0940625" y2="8.740625" width="0" layer="19" extent="1-1"/>
+<wire x1="14.8940625" y1="5.540625" x2="15.9940625" y2="5.440625" width="0" layer="19" extent="1-1"/>
+<wire x1="16.8734375" y1="15.954375" x2="14.8940625" y2="9.540625" width="0" layer="19" extent="1-1"/>
 <wire x1="9.06375" y1="14.5834375" x2="14.8940625" y2="9.540625" width="0" layer="19" extent="1-1"/>
 <wire x1="7.76375" y1="12.4834375" x2="9.06375" y2="14.5834375" width="0" layer="19" extent="1-1"/>
 <wire x1="6.749375" y1="19.2844375" x2="9.06375" y2="14.5834375" width="0" layer="19" extent="1-1"/>
-<wire x1="4.994375" y1="29.5275" x2="6.749375" y2="19.2844375" width="0" layer="19" extent="1-1"/>
-<wire x1="5.2325" y1="32.0675" x2="4.994375" y2="29.5275" width="0" layer="19" extent="1-1"/>
-<wire x1="5.3515625" y1="35.163125" x2="5.2325" y2="32.0675" width="0" layer="19" extent="1-1"/>
-<wire x1="16.8734375" y1="15.954375" x2="7.76375" y2="12.4834375" width="0" layer="19" extent="1-1"/>
 <wire x1="16.3971875" y1="26.3128125" x2="16.8734375" y2="15.954375" width="0" layer="19" extent="1-1"/>
 <wire x1="15.9209375" y1="29.9640625" x2="16.3971875" y2="26.3128125" width="0" layer="19" extent="1-1"/>
 <wire x1="15.7225" y1="40.1240625" x2="15.9209375" y2="29.9640625" width="0" layer="19" extent="1-1"/>
 <wire x1="6.753125" y1="38.8540625" x2="15.7225" y2="40.1240625" width="0" layer="19" extent="1-1"/>
-</signal>
-<signal name="MISO">
-<contactref element="IC3" pad="GPIO12"/>
-<contactref element="IC4" pad="12"/>
-<wire x1="17.0940625" y1="8.740625" x2="22.2959375" y2="10.4290625" width="0" layer="19" extent="1-1"/>
-</signal>
-<signal name="MOSI">
-<contactref element="IC3" pad="GPIO13"/>
-<contactref element="IC4" pad="13"/>
-<wire x1="17.0940625" y1="9.540625" x2="22.2959375" y2="8.4290625" width="0" layer="19" extent="1-1"/>
-</signal>
-<signal name="SCK">
-<contactref element="IC3" pad="GPIO14"/>
-<contactref element="IC4" pad="14"/>
-<wire x1="15.9940625" y1="9.640625" x2="22.2959375" y2="12.4290625" width="0" layer="19" extent="1-1"/>
+<wire x1="5.3515625" y1="35.163125" x2="6.753125" y2="38.8540625" width="0" layer="19" extent="1-1"/>
+<wire x1="5.2325" y1="32.0675" x2="5.3515625" y2="35.163125" width="0" layer="19" extent="1-1"/>
+<wire x1="4.994375" y1="29.5275" x2="5.2325" y2="32.0675" width="0" layer="19" extent="1-1"/>
+<wire x1="23.898125" y1="34.8853125" x2="14.8940625" y2="5.540625" width="0" layer="19" extent="1-1"/>
+<wire x1="24.374375" y1="38.338125" x2="23.898125" y2="34.8853125" width="0" layer="19" extent="1-1"/>
 </signal>
 <signal name="GPIO0">
@@
 <wire x1="5.153125" y1="38.8540625" x2="22.2959375" y2="16.4290625" width="0" layer="19" extent="1-1"/>
 </signal>
-<signal name="!ACC_CS">
-<contactref element="IC4" pad="7"/>
-<contactref element="IC3" pad="GPIO16"/>
-<wire x1="15.9940625" y1="5.440625" x2="22.2959375" y2="14.4290625" width="0" layer="19" extent="1-1"/>
-</signal>
 <signal name="ACC_INT1">
 <contactref element="IC4" pad="8"/>
-<contactref element="IC3" pad="GPIO4"/>
-<wire x1="17.0940625" y1="5.540625" x2="39.6959375" y2="14.4290625" width="0" layer="19" extent="1-1"/>
+<contactref element="J3" pad="1"/>
+<wire x1="57.785" y1="9.604375" x2="17.0940625" y2="5.540625" width="0" layer="19" extent="1-1"/>
 </signal>
 <signal name="ACC_INT2">
 <contactref element="IC4" pad="9"/>
-<contactref element="IC3" pad="GPIO5"/>
-<wire x1="17.0940625" y1="6.340625" x2="39.6959375" y2="16.4290625" width="0" layer="19" extent="1-1"/>
+<contactref element="J3" pad="2"/>
+<wire x1="57.785" y1="12.144375" x2="17.0940625" y2="6.340625" width="0" layer="19" extent="1-1"/>
 </signal>
 <signal name="N$7">
@@
 <wire x1="16.51625" y1="12.938125" x2="15.2734375" y2="15.954375" width="0" layer="19" extent="1-1"/>
 </signal>
+<signal name="SDA">
+<contactref element="IC3" pad="GPIO4"/>
+<contactref element="IC4" pad="13"/>
+<contactref element="R10" pad="1"/>
+<wire x1="17.0940625" y1="9.540625" x2="39.6959375" y2="14.4290625" width="0" layer="19" extent="1-1"/>
+<wire x1="22.774375" y1="38.338125" x2="17.0940625" y2="9.540625" width="0" layer="19" extent="1-1"/>
+</signal>
+<signal name="SCL">
+<contactref element="IC3" pad="GPIO5"/>
+<contactref element="IC4" pad="14"/>
+<contactref element="R11" pad="1"/>
+<wire x1="15.9940625" y1="9.640625" x2="39.6959375" y2="16.4290625" width="0" layer="19" extent="1-1"/>
+<wire x1="22.298125" y1="34.8853125" x2="15.9940625" y2="9.640625" width="0" layer="19" extent="1-1"/>
+</signal>
+<signal name="GPIO16">
+<contactref element="IC3" pad="GPIO16"/>
+<contactref element="J2" pad="4"/>
+<wire x1="52.784375" y1="15.71625" x2="22.2959375" y2="14.4290625" width="0" layer="19" extent="1-1"/>
+</signal>
+<signal name="GPIO14">
+<contactref element="IC3" pad="GPIO14"/>
+<contactref element="J2" pad="3"/>
+<wire x1="52.784375" y1="13.17625" x2="22.2959375" y2="12.4290625" width="0" layer="19" extent="1-1"/>
+</signal>
+<signal name="GPIO13">
+<contactref element="IC3" pad="GPIO13"/>
+<contactref element="J2" pad="2"/>
+<wire x1="52.784375" y1="10.63625" x2="22.2959375" y2="8.4290625" width="0" layer="19" extent="1-1"/>
+</signal>
+<signal name="GPIO12">
+<contactref element="IC3" pad="GPIO12"/>
+<contactref element="J2" pad="1"/>
+<wire x1="52.784375" y1="8.09625" x2="22.2959375" y2="10.4290625" width="0" layer="19" extent="1-1"/>
+</signal>
 </signals>

Commit message: foo
Parts:
- removed R5: 10kΩ, freetronics-luke:0603
- added R12: 10kΩ, freetronics-luke:0603
Connections:
- new net N$1: IC1.1, IC1.4, R4.2
- net +3.3V: no longer R4.2
- net ADC: now also R12.2; no longer IC1.1, IC1.4, R5.2
- net GND: now also R12.1; no longer R5.1
Changed lines of the file:
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@@
 <attribute name="PACKAGE" value="0603" x="16.1528125" y="19.52625" size="0.4064" layer="27" display="off"/>
-</element>
-<element name="R5" library="freetronics-luke" package="0603" value="10kΩ" x="16.4703125" y="22.463125">
-<attribute name="PACKAGE" value="0603" x="16.4703125" y="22.463125" size="0.4064" layer="27" display="off"/>
 </element>
 <element name="R4" library="freetronics-luke" package="0603" value="10kΩ" x="15.5971875" y="26.3128125">
@@
 <element name="R10" library="freetronics-luke" package="0603" value="4.7kΩ" x="23.574375" y="38.338125">
 <attribute name="PACKAGE" value="0603" x="23.574375" y="38.338125" size="0.4064" layer="27" display="off"/>
+</element>
+<element name="R12" library="freetronics-luke" package="0603" value="10kΩ" x="2.38125" y="0.9525">
+<attribute name="PACKAGE" value="0603" x="2.38125" y="0.9525" size="0.4064" layer="27" display="off"/>
 </element>
 </elements>
@@
 <contactref element="J1" pad="3"/>
 <contactref element="R3" pad="1"/>
-<contactref element="R5" pad="1"/>
 <contactref element="R8" pad="1"/>
+<contactref element="R12" pad="1"/>
 <wire x1="46.4740625" y1="10.95375" x2="46.4740625" y2="13.49375" width="0" layer="19" extent="1-1"/>
 <wire x1="39.6959375" y1="6.4290625" x2="46.4740625" y2="10.95375" width="0" layer="19" extent="1-1"/>
@@
 <wire x1="14.8940625" y1="7.140625" x2="14.8940625" y2="6.340625" width="0" layer="19" extent="1-1"/>
 <wire x1="14.8940625" y1="8.740625" x2="14.8940625" y2="7.140625" width="0" layer="19" extent="1-1"/>
+<wire x1="14.91625" y1="12.938125" x2="14.8940625" y2="8.740625" width="0" layer="19" extent="1-1"/>
 <wire x1="10.04875" y1="8.6096875" x2="14.8940625" y2="8.740625" width="0" layer="19" extent="1-1"/>
 <wire x1="8.41375" y1="12.4834375" x2="10.04875" y2="8.6096875" width="0" layer="19" extent="1-1"/>
 <wire x1="7.699375" y1="16.6724375" x2="8.41375" y2="12.4834375" width="0" layer="19" extent="1-1"/>
+<wire x1="1.58125" y1="0.9525" x2="10.04875" y2="8.6096875" width="0" layer="19" extent="1-1"/>
 <wire x1="6.594375" y1="29.5275" x2="7.699375" y2="16.6724375" width="0" layer="19" extent="1-1"/>
 <wire x1="6.8325" y1="32.0675" x2="6.594375" y2="29.5275" width="0" layer="19" extent="1-1"/>
 <wire x1="6.9515625" y1="35.163125" x2="6.8325" y2="32.0675" width="0" layer="19" extent="1-1"/>
-<wire x1="14.91625" y1="12.938125" x2="10.04875" y2="8.6096875" width="0" layer="19" extent="1-1"/>
-<wire x1="15.6703125" y1="22.463125" x2="14.91625" y2="12.938125" width="0" layer="19" extent="1-1"/>
-<wire x1="14.7178125" y1="35.1234375" x2="15.6703125" y2="22.463125" width="0" layer="19" extent="1-1"/>
+<wire x1="14.7178125" y1="35.1234375" x2="6.9515625" y2="35.163125" width="0" layer="19" extent="1-1"/>
 </signal>
 <signal name="+3.3V">
@@
 <contactref element="IC1" pad="5"/>
 <contactref element="J1" pad="1"/>
-<contactref element="R4" pad="2"/>
 <contactref element="R6" pad="2"/>
 <contactref element="R7" pad="2"/>
@@
 <contactref element="R10" pad="2"/>
 <contactref element="R11" pad="2"/>
-<wire x1="22.2959375" y1="6.4290625" x2="46.4740625" y2="8.41375" width="0" layer="19" extent="1-1"/>
-<wire x1="17.0940625" y1="8.740625" x2="22.2959375" y2="6.4290625" width="0" layer="19" extent="1-1"/>
-<wire x1="14.8940625" y1="9.540625" x2="17.0940625" y2="8.740625" width="0" layer="19" extent="1-1"/>
-<wire x1="15.9940625" y1="5.440625" x2="17.0940625" y2="8.740625" width="0" layer="19" extent="1-1"/>
-<wire x1="14.8940625" y1="5.540625" x2="15.9940625" y2="5.440625" width="0" layer="19" extent="1-1"/>
-<wire x1="16.8734375" y1="15.954375" x2="14.8940625" y2="9.540625" width="0" layer="19" extent="1-1"/>
-<wire x1="9.06375" y1="14.5834375" x2="14.8940625" y2="9.540625" width="0" layer="19" extent="1-1"/>
-<wire x1="7.76375" y1="12.4834375" x2="9.06375" y2="14.5834375" width="0" layer="19" extent="1-1"/>
-<wire x1="6.749375" y1="19.2844375" x2="9.06375" y2="14.5834375" width="0" layer="19" extent="1-1"/>
-<wire x1="16.3971875" y1="26.3128125" x2="16.8734375" y2="15.954375" width="0" layer="19" extent="1-1"/>
-<wire x1="15.9209375" y1="29.9640625" x2="16.3971875" y2="26.3128125" width="0" layer="19" extent="1-1"/>
-<wire x1="15.7225" y1="40.1240625" x2="15.9209375" y2="29.9640625" width="0" layer="19" extent="1-1"/>
+<wire x1="23.898125" y1="34.8853125" x2="24.374375" y2="38.338125" width="0" layer="19" extent="1-1"/>
+<wire x1="15.7225" y1="40.1240625" x2="24.374375" y2="38.338125" width="0" layer="19" extent="1-1"/>
 <wire x1="6.753125" y1="38.8540625" x2="15.7225" y2="40.1240625" width="0" layer="19" extent="1-1"/>
 <wire x1="5.3515625" y1="35.163125" x2="6.753125" y2="38.8540625" width="0" layer="19" extent="1-1"/>
 <wire x1="5.2325" y1="32.0675" x2="5.3515625" y2="35.163125" width="0" layer="19" extent="1-1"/>
 <wire x1="4.994375" y1="29.5275" x2="5.2325" y2="32.0675" width="0" layer="19" extent="1-1"/>
-<wire x1="23.898125" y1="34.8853125" x2="14.8940625" y2="5.540625" width="0" layer="19" extent="1-1"/>
-<wire x1="24.374375" y1="38.338125" x2="23.898125" y2="34.8853125" width="0" layer="19" extent="1-1"/>
+<wire x1="15.9209375" y1="29.9640625" x2="23.898125" y2="34.8853125" width="0" layer="19" extent="1-1"/>
+<wire x1="6.749375" y1="19.2844375" x2="4.994375" y2="29.5275" width="0" layer="19" extent="1-1"/>
+<wire x1="9.06375" y1="14.5834375" x2="6.749375" y2="19.2844375" width="0" layer="19" extent="1-1"/>
+<wire x1="7.76375" y1="12.4834375" x2="9.06375" y2="14.5834375" width="0" layer="19" extent="1-1"/>
+<wire x1="14.8940625" y1="9.540625" x2="9.06375" y2="14.5834375" width="0" layer="19" extent="1-1"/>
+<wire x1="17.0940625" y1="8.740625" x2="14.8940625" y2="9.540625" width="0" layer="19" extent="1-1"/>
+<wire x1="15.9940625" y1="5.440625" x2="17.0940625" y2="8.740625" width="0" layer="19" extent="1-1"/>
+<wire x1="14.8940625" y1="5.540625" x2="15.9940625" y2="5.440625" width="0" layer="19" extent="1-1"/>
+<wire x1="22.2959375" y1="6.4290625" x2="17.0940625" y2="8.740625" width="0" layer="19" extent="1-1"/>
+<wire x1="16.8734375" y1="15.954375" x2="14.8940625" y2="9.540625" width="0" layer="19" extent="1-1"/>
+<wire x1="46.4740625" y1="8.41375" x2="22.2959375" y2="6.4290625" width="0" layer="19" extent="1-1"/>
 </signal>
 <signal name="GPIO0">
@@
 <signal name="ADC">
 <contactref element="IC3" pad="ADC"/>
-<contactref element="IC1" pad="4"/>
-<contactref element="IC1" pad="1"/>
 <contactref element="C2" pad="2"/>
-<contactref element="R5" pad="2"/>
 <contactref element="R4" pad="1"/>
-<wire x1="8.649375" y1="19.2844375" x2="22.2959375" y2="18.4290625" width="0" layer="19" extent="1-1"/>
-<wire x1="6.749375" y1="16.6724375" x2="8.649375" y2="19.2844375" width="0" layer="19" extent="1-1"/>
-<wire x1="7.705625" y1="23.415625" x2="8.649375" y2="19.2844375" width="0" layer="19" extent="1-1"/>
-<wire x1="17.2703125" y1="22.463125" x2="6.749375" y2="16.6724375" width="0" layer="19" extent="1-1"/>
-<wire x1="14.7971875" y1="26.3128125" x2="17.2703125" y2="22.463125" width="0" layer="19" extent="1-1"/>
+<contactref element="R12" pad="2"/>
+<wire x1="14.7971875" y1="26.3128125" x2="22.2959375" y2="18.4290625" width="0" layer="19" extent="1-1"/>
+<wire x1="7.705625" y1="23.415625" x2="14.7971875" y2="26.3128125" width="0" layer="19" extent="1-1"/>
+<wire x1="3.18125" y1="0.9525" x2="7.705625" y2="23.415625" width="0" layer="19" extent="1-1"/>
 </signal>
 <signal name="GPIO3">
@@
 <wire x1="52.784375" y1="8.09625" x2="22.2959375" y2="10.4290625" width="0" layer="19" extent="1-1"/>
 </signal>
+<signal name="N$1">
+<contactref element="IC1" pad="4"/>
+<contactref element="IC1" pad="1"/>
+<contactref element="R4" pad="2"/>
+<wire x1="8.649375" y1="19.2844375" x2="16.3971875" y2="26.3128125" width="0" layer="19" extent="1-1"/>
+<wire x1="6.749375" y1="16.6724375" x2="8.649375" y2="19.2844375" width="0" layer="19" extent="1-1"/>
+</signal>
 </signals>
