File: thingy.brd (EAGLE design)
At the start: 24 parts, among them IC1 MCP6001T-I/OT, IC2 MAX9812LEXT+T, IC3 ESP-12, IC4 ADXL345BCCZ, J1 Interface, J2 GPIO, J3 Interrupts, Q1 Electret Mic

Commit message: foo
Parts:
- moved R12 25.3 mm to (15.8, 22.4)
- moved R10 17.2 mm to (6.47, 39.6)
- moved R11 8.62 mm to (15.2, 38.4)
- moved R7 4.54 mm to (15.3, 35.6)
- moved R8 2.28 mm to (15.2, 32.9)
- moved R9 1.51 mm to (6.07, 37.3)
Changed lines of the file:
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@@
 <attribute name="PACKAGE" value="0603" x="15.1209375" y="29.9640625" size="0.4064" layer="27" display="off"/>
 </element>
-<element name="R7" library="freetronics-luke" package="0603" value="10kΩ" x="14.9225" y="40.1240625">
-<attribute name="PACKAGE" value="0603" x="14.9225" y="40.1240625" size="0.4064" layer="27" display="off"/>
+<element name="R7" library="freetronics-luke" package="0603" value="10kΩ" x="15.2796875" y="35.5996875">
+<attribute name="PACKAGE" value="0603" x="15.2796875" y="35.5996875" size="0.4064" layer="27" display="off"/>
 </element>
-<element name="R9" library="freetronics-luke" package="0603" value="10kΩ" x="5.953125" y="38.8540625">
-<attribute name="PACKAGE" value="0603" x="5.953125" y="38.8540625" size="0.4064" layer="27" display="off"/>
+<element name="R9" library="freetronics-luke" package="0603" value="10kΩ" x="6.0721875" y="37.3459375">
+<attribute name="PACKAGE" value="0603" x="6.0721875" y="37.3459375" size="0.4064" layer="27" display="off"/>
 </element>
-<element name="R8" library="freetronics-luke" package="0603" value="10kΩ" x="15.5178125" y="35.1234375">
-<attribute name="PACKAGE" value="0603" x="15.5178125" y="35.1234375" size="0.4064" layer="27" display="off"/>
+<element name="R8" library="freetronics-luke" package="0603" value="10kΩ" x="15.2003125" y="32.86125">
+<attribute name="PACKAGE" value="0603" x="15.2003125" y="32.86125" size="0.4064" layer="27" display="off"/>
 </element>
 <element name="J3" library="pinhead" package="1X02" value="Interrupts" x="57.785" y="10.874375" rot="R90"/>
 <element name="J2" library="pinhead" package="1X04" value="GPIO" x="52.784375" y="11.90625" rot="R90"/>
-<element name="R11" library="freetronics-luke" package="0603" value="4.7kΩ" x="23.098125" y="34.8853125">
-<attribute name="PACKAGE" value="0603" x="23.098125" y="34.8853125" size="0.4064" layer="27" display="off"/>
+<element name="R11" library="freetronics-luke" package="0603" value="4.7kΩ" x="15.24" y="38.4175">
+<attribute name="PACKAGE" value="0603" x="15.24" y="38.4175" size="0.4064" layer="27" display="off"/>
 </element>
-<element name="R10" library="freetronics-luke" package="0603" value="4.7kΩ" x="23.574375" y="38.338125">
-<attribute name="PACKAGE" value="0603" x="23.574375" y="38.338125" size="0.4064" layer="27" display="off"/>
+<element name="R10" library="freetronics-luke" package="0603" value="4.7kΩ" x="6.4690625" y="39.608125">
+<attribute name="PACKAGE" value="0603" x="6.4690625" y="39.608125" size="0.4064" layer="27" display="off"/>
 </element>
-<element name="R12" library="freetronics-luke" package="0603" value="10kΩ" x="2.38125" y="0.9525">
-<attribute name="PACKAGE" value="0603" x="2.38125" y="0.9525" size="0.4064" layer="27" display="off"/>
+<element name="R12" library="freetronics-luke" package="0603" value="10kΩ" x="15.8353125" y="22.38375">
+<attribute name="PACKAGE" value="0603" x="15.8353125" y="22.38375" size="0.4064" layer="27" display="off"/>
 </element>
 </elements>
@@
 <wire x1="8.41375" y1="12.4834375" x2="10.04875" y2="8.6096875" width="0" layer="19" extent="1-1"/>
 <wire x1="7.699375" y1="16.6724375" x2="8.41375" y2="12.4834375" width="0" layer="19" extent="1-1"/>
-<wire x1="1.58125" y1="0.9525" x2="10.04875" y2="8.6096875" width="0" layer="19" extent="1-1"/>
+<wire x1="15.0353125" y1="22.38375" x2="10.04875" y2="8.6096875" width="0" layer="19" extent="1-1"/>
 <wire x1="6.594375" y1="29.5275" x2="7.699375" y2="16.6724375" width="0" layer="19" extent="1-1"/>
 <wire x1="6.8325" y1="32.0675" x2="6.594375" y2="29.5275" width="0" layer="19" extent="1-1"/>
 <wire x1="6.9515625" y1="35.163125" x2="6.8325" y2="32.0675" width="0" layer="19" extent="1-1"/>
-<wire x1="14.7178125" y1="35.1234375" x2="6.9515625" y2="35.163125" width="0" layer="19" extent="1-1"/>
+<wire x1="14.4003125" y1="32.86125" x2="6.9515625" y2="35.163125" width="0" layer="19" extent="1-1"/>
 </signal>
 <signal name="+3.3V">
@@
 <contactref element="R10" pad="2"/>
 <contactref element="R11" pad="2"/>
-<wire x1="23.898125" y1="34.8853125" x2="24.374375" y2="38.338125" width="0" layer="19" extent="1-1"/>
-<wire x1="15.7225" y1="40.1240625" x2="24.374375" y2="38.338125" width="0" layer="19" extent="1-1"/>
-<wire x1="6.753125" y1="38.8540625" x2="15.7225" y2="40.1240625" width="0" layer="19" extent="1-1"/>
-<wire x1="5.3515625" y1="35.163125" x2="6.753125" y2="38.8540625" width="0" layer="19" extent="1-1"/>
+<wire x1="16.04" y1="38.4175" x2="7.2690625" y2="39.608125" width="0" layer="19" extent="1-1"/>
+<wire x1="16.0796875" y1="35.5996875" x2="7.2690625" y2="39.608125" width="0" layer="19" extent="1-1"/>
+<wire x1="6.8721875" y1="37.3459375" x2="16.0796875" y2="35.5996875" width="0" layer="19" extent="1-1"/>
+<wire x1="5.3515625" y1="35.163125" x2="6.8721875" y2="37.3459375" width="0" layer="19" extent="1-1"/>
 <wire x1="5.2325" y1="32.0675" x2="5.3515625" y2="35.163125" width="0" layer="19" extent="1-1"/>
 <wire x1="4.994375" y1="29.5275" x2="5.2325" y2="32.0675" width="0" layer="19" extent="1-1"/>
-<wire x1="15.9209375" y1="29.9640625" x2="23.898125" y2="34.8853125" width="0" layer="19" extent="1-1"/>
+<wire x1="15.9209375" y1="29.9640625" x2="16.04" y2="38.4175" width="0" layer="19" extent="1-1"/>
 <wire x1="6.749375" y1="19.2844375" x2="4.994375" y2="29.5275" width="0" layer="19" extent="1-1"/>
 <wire x1="9.06375" y1="14.5834375" x2="6.749375" y2="19.2844375" width="0" layer="19" extent="1-1"/>
@@
 <contactref element="IC3" pad="RST"/>
 <contactref element="R7" pad="1"/>
-<wire x1="14.1225" y1="40.1240625" x2="22.2959375" y2="20.4290625" width="0" layer="19" extent="1-1"/>
+<wire x1="14.4796875" y1="35.5996875" x2="22.2959375" y2="20.4290625" width="0" layer="19" extent="1-1"/>
 </signal>
 <signal name="CHPD">
 <contactref element="IC3" pad="CHPD"/>
 <contactref element="R9" pad="1"/>
-<wire x1="5.153125" y1="38.8540625" x2="22.2959375" y2="16.4290625" width="0" layer="19" extent="1-1"/>
+<wire x1="5.2721875" y1="37.3459375" x2="22.2959375" y2="16.4290625" width="0" layer="19" extent="1-1"/>
 </signal>
 <signal name="ACC_INT1">
@@
 <contactref element="IC3" pad="GPIO15"/>
 <contactref element="R8" pad="2"/>
-<wire x1="16.3178125" y1="35.1234375" x2="39.6959375" y2="8.4290625" width="0" layer="19" extent="1-1"/>
+<wire x1="16.0003125" y1="32.86125" x2="39.6959375" y2="8.4290625" width="0" layer="19" extent="1-1"/>
 </signal>
 <signal name="N$13">
@@
 <wire x1="14.7971875" y1="26.3128125" x2="22.2959375" y2="18.4290625" width="0" layer="19" extent="1-1"/>
 <wire x1="7.705625" y1="23.415625" x2="14.7971875" y2="26.3128125" width="0" layer="19" extent="1-1"/>
-<wire x1="3.18125" y1="0.9525" x2="7.705625" y2="23.415625" width="0" layer="19" extent="1-1"/>
+<wire x1="16.6353125" y1="22.38375" x2="7.705625" y2="23.415625" width="0" layer="19" extent="1-1"/>
 </signal>
 <signal name="GPIO3">
@@
 <contactref element="R10" pad="1"/>
 <wire x1="17.0940625" y1="9.540625" x2="39.6959375" y2="14.4290625" width="0" layer="19" extent="1-1"/>
-<wire x1="22.774375" y1="38.338125" x2="17.0940625" y2="9.540625" width="0" layer="19" extent="1-1"/>
+<wire x1="5.6690625" y1="39.608125" x2="17.0940625" y2="9.540625" width="0" layer="19" extent="1-1"/>
 </signal>
 <signal name="SCL">
@@
 <contactref element="R11" pad="1"/>
 <wire x1="15.9940625" y1="9.640625" x2="39.6959375" y2="16.4290625" width="0" layer="19" extent="1-1"/>
-<wire x1="22.298125" y1="34.8853125" x2="15.9940625" y2="9.640625" width="0" layer="19" extent="1-1"/>
+<wire x1="14.44" y1="38.4175" x2="15.9940625" y2="9.640625" width="0" layer="19" extent="1-1"/>
 </signal>
 <signal name="GPIO16">
